Commit message: Modified URDF to make compatible with ROS 2 iron

File: ur_robotiq_description/urdf/robotiq_2f_85_urdf.xacro (robot description, xacro)
@@ -10,12 +10,10 @@
         sim_ignition:=false
         sim_isaac:=false
-        isaac_joint_commands:=/isaac_joint_commands
-        isaac_joint_states:=/isaac_joint_states
         use_fake_hardware:=false
         fake_sensor_commands:=false
-        include_ros2_control:=false
+        include_ros2_control:=true
         com_port:=/dev/ttyUSB0">
         <!-- ros2 control include -->
-        <xacro:include filename="$(find robotiq_description)/urdf/2f_85.ros2_control.xacro" />
+        <xacro:include filename="$(find robotiq_description)/urdf/robotiq_gripper.ros2_control.xacro" />
         <!-- if we are simulating or directly communicating with the gripper we need a ros2 control instance -->
         <xacro:if value="${include_ros2_control}">
@@ -24,6 +22,4 @@
                 sim_ignition="${sim_ignition}"
                 sim_isaac="${sim_isaac}"
-                isaac_joint_commands="${isaac_joint_commands}"
-                isaac_joint_states="${isaac_joint_states}"
                 use_fake_hardware="${use_fake_hardware}"
                 fake_sensor_commands="${fake_sensor_commands}"
@@ -33,10 +29,10 @@
             <visual>
                 <geometry>
-                    <mesh filename="file://$(find robotiq_description)/meshes/visual/2f_85/robotiq_base.dae" />
-                </geometry>
-            </visual>
-            <collision>
-                <geometry>
-                    <mesh filename="file://$(find robotiq_description)/meshes/collision/2f_85/robotiq_base.stl" />
+                    <mesh filename="file://$(find robotiq_description)/meshes/visual/robotiq_base.dae" />
+                </geometry>
+            </visual>
+            <collision>
+                <geometry>
+                    <mesh filename="file://$(find robotiq_description)/meshes/collision/robotiq_base.stl" />
                 </geometry>
             </collision>
@@ -50,10 +46,10 @@
             <visual>
                 <geometry>
-                    <mesh filename="file://$(find robotiq_description)/meshes/visual/2f_85/left_knuckle.dae" />
-                </geometry>
-            </visual>
-            <collision>
-                <geometry>
-                    <mesh filename="file://$(find robotiq_description)/meshes/collision/2f_85/left_knuckle.stl" />
+                    <mesh filename="file://$(find robotiq_description)/meshes/visual/left_knuckle.dae" />
+                </geometry>
+            </visual>
+            <collision>
+                <geometry>
+                    <mesh filename="file://$(find robotiq_description)/meshes/collision/left_knuckle.stl" />
                 </geometry>
             </collision>
@@ -67,10 +63,10 @@
             <visual>
                 <geometry>
-                    <mesh filename="file://$(find robotiq_description)/meshes/visual/2f_85/right_knuckle.dae" />
-                </geometry>
-            </visual>
-            <collision>
-                <geometry>
-                    <mesh filename="file://$(find robotiq_description)/meshes/collision/2f_85/right_knuckle.stl" />
+                    <mesh filename="file://$(find robotiq_description)/meshes/visual/right_knuckle.dae" />
+                </geometry>
+            </visual>
+            <collision>
+                <geometry>
+                    <mesh filename="file://$(find robotiq_description)/meshes/collision/right_knuckle.stl" />
                 </geometry>
             </collision>
@@ -84,10 +80,10 @@
             <visual>
                 <geometry>
-                    <mesh filename="file://$(find robotiq_description)/meshes/visual/2f_85/left_finger.dae" />
-                </geometry>
-            </visual>
-            <collision>
-                <geometry>
-                    <mesh filename="file://$(find robotiq_description)/meshes/collision/2f_85/left_finger.stl" />
+                    <mesh filename="file://$(find robotiq_description)/meshes/visual/left_finger.dae" />
+                </geometry>
+            </visual>
+            <collision>
+                <geometry>
+                    <mesh filename="file://$(find robotiq_description)/meshes/collision/left_finger.stl" />
                 </geometry>
             </collision>
@@ -101,10 +97,10 @@
             <visual>
                 <geometry>
-                    <mesh filename="file://$(find robotiq_description)/meshes/visual/2f_85/right_finger.dae" />
-                </geometry>
-            </visual>
-            <collision>
-                <geometry>
-                    <mesh filename="file://$(find robotiq_description)/meshes/collision/2f_85/right_finger.stl" />
+                    <mesh filename="file://$(find robotiq_description)/meshes/visual/right_finger.dae" />
+                </geometry>
+            </visual>
+            <collision>
+                <geometry>
+                    <mesh filename="file://$(find robotiq_description)/meshes/collision/right_finger.stl" />
                 </geometry>
             </collision>
@@ -118,10 +114,10 @@
             <visual>
                 <geometry>
-                    <mesh filename="file://$(find robotiq_description)/meshes/visual/2f_85/left_inner_knuckle.dae" />
-                </geometry>
-            </visual>
-            <collision>
-                <geometry>
-                    <mesh filename="file://$(find robotiq_description)/meshes/collision/2f_85/left_inner_knuckle.stl" />
+                    <mesh filename="file://$(find robotiq_description)/meshes/visual/left_inner_knuckle.dae" />
+                </geometry>
+            </visual>
+            <collision>
+                <geometry>
+                    <mesh filename="file://$(find robotiq_description)/meshes/collision/left_inner_knuckle.stl" />
                 </geometry>
             </collision>
@@ -135,10 +131,10 @@
             <visual>
                 <geometry>
-                    <mesh filename="file://$(find robotiq_description)/meshes/visual/2f_85/right_inner_knuckle.dae" />
-                </geometry>
-            </visual>
-            <collision>
-                <geometry>
-                    <mesh filename="file://$(find robotiq_description)/meshes/collision/2f_85/right_inner_knuckle.stl" />
+                    <mesh filename="file://$(find robotiq_description)/meshes/visual/right_inner_knuckle.dae" />
+                </geometry>
+            </visual>
+            <collision>
+                <geometry>
+                    <mesh filename="file://$(find robotiq_description)/meshes/collision/right_inner_knuckle.stl" />
                 </geometry>
             </collision>
@@ -152,10 +148,10 @@
             <visual>
                 <geometry>
-                    <mesh filename="file://$(find robotiq_description)/meshes/visual/2f_85/left_finger_tip.dae" />
-                </geometry>
-            </visual>
-            <collision>
-                <geometry>
-                    <mesh filename="file://$(find robotiq_description)/meshes/collision/2f_85/left_finger_tip.stl" />
+                    <mesh filename="file://$(find robotiq_description)/meshes/visual/left_finger_tip.dae" />
+                </geometry>
+            </visual>
+            <collision>
+                <geometry>
+                    <mesh filename="file://$(find robotiq_description)/meshes/collision/left_finger_tip.stl" />
                 </geometry>
                 <surface>
@@ -187,10 +183,10 @@
             <visual>
                 <geometry>
-                    <mesh filename="file://$(find robotiq_description)/meshes/visual/2f_85/right_finger_tip.dae" />
-                </geometry>
-            </visual>
-            <collision>
-                <geometry>
-                    <mesh filename="file://$(find robotiq_description)/meshes/collision/2f_85/right_finger_tip.stl" />
+                    <mesh filename="file://$(find robotiq_description)/meshes/visual/right_finger_tip.dae" />
+                </geometry>
+            </visual>
+            <collision>
+                <geometry>
+                    <mesh filename="file://$(find robotiq_description)/meshes/collision/right_finger_tip.stl" />
                 </geometry>
                 <surface>

Commit message: Parameterized Xacro for UR3e

File: ur_robotiq_description/urdf/robotiq_2f_85_urdf.xacro (robot description, xacro)
@@ -3,4 +3,6 @@
     <!-- parameters -->
     <xacro:arg name="use_fake_hardware" default="true" />
+    <!-- If visualizing just the gripper with no arm, set the true, otherwise, set to false -->
+    <xacro:property name="gripper_only" value="false"/>
     <xacro:macro name="robotiq_gripper" params="
         name
@@ -274,13 +276,14 @@
         </joint>
     </xacro:macro>
-    <!-- Uncomment this block if you want to see only the gripper in RViz
-    <link name="world" />
-    <xacro:robotiq_gripper name="RobotiqGripperHardwareInterface" prefix="" parent="world" use_fake_hardware="$(arg use_fake_hardware)">
-        <origin xyz="0 0 0" rpy="0 0 0" />
-    </xacro:robotiq_gripper>
-     -->
-    <!-- Uncomment this block if you want to see the UR3e with the Robotiq 2F-85 attached. -->
-    <xacro:robotiq_gripper name="RobotiqGripperHardwareInterface" prefix="" parent="ur3e_tool0" use_fake_hardware="$(arg use_fake_hardware)">
-        <origin xyz="0 0 0" rpy="0 0 0" />
-    </xacro:robotiq_gripper>
+    <xacro:if value="${gripper_only}">
+    	<link name="world" />
+    	<xacro:robotiq_gripper name="RobotiqGripperHardwareInterface" prefix="" parent="world" use_fake_hardware="$(arg use_fake_hardware)">
+        	<origin xyz="0 0 0" rpy="0 0 0" />
+    	</xacro:robotiq_gripper>
+    </xacro:if>
+    <xacro:if value="${not gripper_only}">
+    	<xacro:robotiq_gripper name="RobotiqGripperHardwareInterface" prefix="" parent="ur3e_tool0" use_fake_hardware="$(arg use_fake_hardware)">
+        	<origin xyz="0 0 0" rpy="0 0 0" />
+    	</xacro:robotiq_gripper>
+    </xacro:if>
 </robot>
